File: mcu.kicad_sch (KiCad schematic)
At the start: 50 parts, among them J101 switch, J3 TYPE-C-31-M-12, Q1 2N7002VC-7, Q2 2N7002VC-7, U101 W25Q128JVPIQ, U102 RP2040, U103 XC6210B332MR-G, Y101 12MHz

Commit message: Cleanup routing
Parts:
- removed TP1: RESET, TestPoint:TestPoint_Pad_1.0x1.0mm, symbol Connector:TestPoint
- removed TP3: BOOTSEL, TestPoint:TestPoint_Pad_1.0x1.0mm, symbol Connector:TestPoint
Connections:
- net ROW-1: now also U102.14 (GPIO11); no longer U102.12 (GPIO9)
- net ROW-3: now also U102.12 (GPIO9); no longer U102.14 (GPIO11)
- net ROW-4: now also U102.11 (GPIO8); no longer U102.29 (GPIO18)
- net ~{BOOTSEL}: now also Q2.3 (D), R15.2
Changed lines of the file:
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@@
   (junction (at 132.334 187.706) (diameter 0) (color 0 0 0 0)
   )
-  (junction (at 263.652 99.695) (diameter 0) (color 0 0 0 0)
-  )
   (junction (at 39.624 88.646) (diameter 0) (color 0 0 0 0)
   )
@@
   (junction (at 218.948 144.78) (diameter 0) (color 0 0 0 0)
   )
-  (junction (at 209.296 85.852) (diameter 0) (color 0 0 0 0)
-  )
   (junction (at 109.474 177.546) (diameter 0) (color 0 0 0 0)
   )
@@
   (no_connect (at 145.288 111.506))
   (no_connect (at 145.034 48.006))
+  (no_connect (at 145.034 83.566))
   (no_connect (at 145.034 88.646))
   (no_connect (at 85.344 106.426))
   (no_connect (at 145.034 45.466))
   (no_connect (at 195.834 35.306))
-  (no_connect (at 145.034 58.166))
   (no_connect (at 145.288 114.046))
   (no_connect (at 145.034 96.266))
@@
     (stroke (width 0) (type default))
   )
-  (wire (pts (xy 141.224 58.166) (xy 145.034 58.166))
-    (stroke (width 0) (type default))
-  )
   (wire (pts (xy 241.3 106.045) (xy 250.952 106.045))
     (stroke (width 0) (type default))
@@
     (stroke (width 0) (type default))
   )
+  (wire (pts (xy 141.224 60.706) (xy 147.574 60.706))
+    (stroke (width 0) (type default))
+  )
   (wire (pts (xy 248.158 142.24) (xy 248.158 144.78))
     (stroke (width 0) (type default))
@@
     (stroke (width 0) (type default))
   )
+  (wire (pts (xy 141.224 58.166) (xy 147.32 58.166))
+    (stroke (width 0) (type default))
+  )
   (wire (pts (xy 38.354 30.226) (xy 35.814 30.226))
     (stroke (width 0) (type default))
@@
     (stroke (width 0) (type default))
   )
-  (wire (pts (xy 209.296 85.852) (xy 218.186 85.852))
-    (stroke (width 0) (type default))
-  )
   (wire (pts (xy 85.09 48.006) (xy 90.424 48.006))
     (stroke (width 0) (type default))
@@
     (stroke (width 0) (type default))
   )
-  (wire (pts (xy 141.224 60.706) (xy 147.574 60.706))
-    (stroke (width 0) (type default))
-  )
   (wire (pts (xy 39.624 120.396) (xy 39.624 125.476))
     (stroke (width 0) (type default))
@@
     (stroke (width 0) (type default))
   )
+  (wire (pts (xy 141.224 65.786) (xy 147.574 65.786))
+    (stroke (width 0) (type default))
+  )
   (polyline (pts (xy 167.64 129.54) (xy 284.988 129.54))
     (stroke (width 0) (type default))
@@
     (stroke (width 0) (type default))
   )
-  (wire (pts (xy 263.652 99.695) (xy 263.652 100.965))
+  (wire (pts (xy 263.652 98.552) (xy 263.652 100.965))
     (stroke (width 0) (type default))
   )
@@
     (stroke (width 0) (type default))
   )
-  (wire (pts (xy 263.652 98.552) (xy 263.652 99.695))
-    (stroke (width 0) (type default))
-  )
   (wire (pts (xy 115.824 124.206) (xy 115.824 121.666))
     (stroke (width 0) (type default))
@@
     (stroke (width 0) (type default))
   )
-  (wire (pts (xy 209.296 83.82) (xy 209.296 85.852))
-    (stroke (width 0) (type default))
-  )
   (wire (pts (xy 78.994 68.326) (xy 90.424 68.326))
     (stroke (width 0) (type default))
@@
     (stroke (width 0) (type default))
   )
-  (wire (pts (xy 209.296 85.852) (xy 209.296 87.63))
-    (stroke (width 0) (type default))
-  )
   (wire (pts (xy 201.422 97.028) (xy 201.422 106.045))
     (stroke (width 0) (type default))
@@
     (stroke (width 0) (type default))
   )
+  (wire (pts (xy 141.224 63.246) (xy 147.574 63.246))
+    (stroke (width 0) (type default))
+  )
   (wire (pts (xy 132.334 186.436) (xy 132.334 187.706))
     (stroke (width 0) (type default))
@@
     (stroke (width 0) (type default))
   )
-  (wire (pts (xy 141.224 83.566) (xy 147.32 83.566))
-    (stroke (width 0) (type default))
-  )
   (wire (pts (xy 162.052 76.454) (xy 162.052 77.47))
     (stroke (width 0) (type default))
@@
     (stroke (width 0) (type default))
   )
-  (wire (pts (xy 141.224 63.246) (xy 147.574 63.246))
-    (stroke (width 0) (type default))
-  )
   (wire (pts (xy 258.064 63.246) (xy 259.334 63.246))
     (stroke (width 0) (type default))
@@
     (stroke (width 0) (type default))
   )
-  (wire (pts (xy 141.224 65.786) (xy 147.574 65.786))
-    (stroke (width 0) (type default))
-  )
   (wire (pts (xy 231.394 32.766) (xy 232.664 32.766))
     (stroke (width 0) (type default))
@@
     (stroke (width 0) (type default))
   )
+  (wire (pts (xy 209.296 83.82) (xy 209.296 87.63))
+    (stroke (width 0) (type default))
+  )
   (wire (pts (xy 86.614 186.436) (xy 86.614 187.706))
     (stroke (width 0) (type default))
@@
     (stroke (width 0) (type default))
   )
+  (wire (pts (xy 141.224 83.566) (xy 145.034 83.566))
+    (stroke (width 0) (type default))
+  )
   (wire (pts (xy 141.224 40.386) (xy 147.574 40.386))
     (stroke (width 0) (type default))
@@
     (stroke (width 0) (type default))
   )
-  (wire (pts (xy 263.652 99.695) (xy 271.272 99.695))
-    (stroke (width 0) (type default))
-  )
   (wire (pts (xy 145.288 111.506) (xy 141.478 111.506))
     (stroke (width 0) (type default))
@@
     (effects (font (size 1.27 1.27)) (justify left bottom))
   )
-  (label "~{RESET}" (at 212.344 85.852 0) (fields_autoplaced)
+  (label "~{RESET}" (at 209.296 86.868 0) (fields_autoplaced)
     (effects (font (size 1.27 1.27)) (justify left bottom))
   )
@@
     (effects (font (size 1.27 1.27)) (justify left bottom))
   )
-  (label "~{BOOTSEL}" (at 264.922 99.568 0) (fields_autoplaced)
+  (label "~{BOOTSEL}" (at 263.652 100.33 0) (fields_autoplaced)
     (effects (font (size 1.27 1.27)) (justify left bottom))
   )
@@
     (effects (font (size 1.27 1.27)) (justify left bottom))
   )
-  (hierarchical_label "ROW-1" (shape input) (at 147.574 60.706 0) (fields_autoplaced)
+  (hierarchical_label "ROW-3" (shape input) (at 147.574 60.706 0) (fields_autoplaced)
     (effects (font (size 1.27 1.27)) (justify left))
   )
-  (hierarchical_label "TX" (shape input) (at 147.574 37.846 0) (fields_autoplaced)
+  (hierarchical_label "ROW-4" (shape input) (at 147.32 58.166 0) (fields_autoplaced)
     (effects (font (size 1.27 1.27)) (justify left))
   )
-  (hierarchical_label "COL-5" (shape input) (at 147.574 78.486 0) (fields_autoplaced)
+  (hierarchical_label "ROW-2" (shape input) (at 147.574 63.246 0) (fields_autoplaced)
     (effects (font (size 1.27 1.27)) (justify left))
   )
-  (hierarchical_label "ROW-4" (shape input) (at 147.32 83.566 0) (fields_autoplaced)
+  (hierarchical_label "TX" (shape input) (at 147.574 37.846 0) (fields_autoplaced)
+    (effects (font (size 1.27 1.27)) (justify left))
+  )
+  (hierarchical_label "COL-5" (shape input) (at 147.574 78.486 0) (fields_autoplaced)
     (effects (font (size 1.27 1.27)) (justify left))
   )
@@
     (effects (font (size 1.27 1.27)) (justify left))
   )
-  (hierarchical_label "ROW-3" (shape input) (at 147.574 65.786 0) (fields_autoplaced)
-    (effects (font (size 1.27 1.27)) (justify left))
-  )
-  (hierarchical_label "ROW-2" (shape input) (at 147.574 63.246 0) (fields_autoplaced)
+  (hierarchical_label "ROW-1" (shape input) (at 147.574 65.786 0) (fields_autoplaced)
     (effects (font (size 1.27 1.27)) (justify left))
   )
@@
     )
   )
-  (symbol (lib_id "Connector:TestPoint") (at 218.186 85.852 270) (unit 1)
-    (in_bom no) (on_board yes) (dnp no)
-    (property "Reference" "TP1" (at 222.631 84.582 90)
-      (effects (font (size 1.27 1.27)) (justify left))
-    )
-    (property "Value" "RESET" (at 222.631 87.122 90)
-      (effects (font (size 1.27 1.27)) (justify left))
-    )
-    (property "Footprint" "TestPoint:TestPoint_Pad_1.0x1.0mm" (at 218.186 90.932 0)
-      (effects (font (size 1.27 1.27)) hide)
-    )
-    (property "Datasheet" "~" (at 218.186 90.932 0)
-      (effects (font (size 1.27 1.27)) hide)
-    )
-    (property "Substitute" "" (at 218.186 85.852 0)
-      (effects (font (size 1.27 1.27)) hide)
-    )
-    (pin "1")
-    (instances
-      (project "sea-picro"
-        (path "/8c6a821f-8e19-48f3-8f44-9b340f7689bc"
-          (reference "TP1") (unit 1)
-        )
-      )
-      (project "Interface"
-        (path "/c9f596c2-7857-4b11-bdf6-e9f4a0e624c2/5c11a847-83df-4611-a1ea-12b908e939bb"
-          (reference "TP1") (unit 1)
-        )
-      )
-    )
-  )
   (symbol (lib_id "Transistor_FET:FDG6335N") (at 214.757 108.585 270) (mirror x) (unit 2)
     (in_bom yes) (on_board yes) (dnp no)
@@
         )
       )
-    )
-  )
-  (symbol (lib_id "Connector:TestPoint") (at 271.272 99.695 270) (unit 1)
-    (in_bom no) (on_board yes) (dnp no)
-    (property "Reference" "TP3" (at 275.717 98.425 90)
-      (effects (font (size 1.27 1.27)) (justify left))
-    )
-    (property "Value" "BOOTSEL" (at 275.717 100.965 90)
-      (effects (font (size 1.27 1.27)) (justify left))
-    )
-    (property "Footprint" "TestPoint:TestPoint_Pad_1.0x1.0mm" (at 271.272 104.775 0)
-      (effects (font (size 1.27 1.27)) hide)
-    )
-    (property "Datasheet" "~" (at 271.272 104.775 0)
-      (effects (font (size 1.27 1.27)) hide)
-    )
-    (property "Substitute" "" (at 271.272 99.695 0)
-      (effects (font (size 1.27 1.27)) hide)
-    )
-    (pin "1")
-    (instances
-      (project "sea-picro"
-        (path "/8c6a821f-8e19-48f3-8f44-9b340f7689bc"
-          (reference "TP3") (unit 1)
-        )
-      )
-      (project "Interface"
-        (path "/c9f596c2-7857-4b11-bdf6-e9f4a0e624c2/5c11a847-83df-4611-a1ea-12b908e939bb"
-          (reference "TP2") (unit 1)
-        )
-      )
