File: mcu.kicad_sch (KiCad schematic)
At the start: 48 parts, among them J101 switch, J3 TYPE-C-31-M-12, Q1 2N7002VC-7, Q2 2N7002VC-7, U101 W25Q128JVPIQ, U102 RP2040, U103 XC6210B332MR-G, Y101 12MHz

Commit message: Complete routing
Connections:
- net COL-1: now also U102.17 (GPIO14); no longer U102.15 (GPIO12)
- net COL-2: now also U102.18 (GPIO15); no longer U102.16 (GPIO13)
- net COL-3: now also U102.27 (GPIO16); no longer U102.17 (GPIO14)
- net COL-4: now also U102.28 (GPIO17); no longer U102.18 (GPIO15)
- net COL-5: now also U102.29 (GPIO18); no longer U102.27 (GPIO16)

Commit message: Rotate and add mirror line
Parts:
- renumbered C109 to C10, C110 to C11, C111 to C12, C112 to C13, C113 to C14, C114 to C15, C115 to C16, C5 to C17, C101 to C2, C102 to C3, C103 to C4, C104 to C5, C105 to C6, C106 to C7, C107 to C8, C108 to C9, D101 to D1, J101 to J102, R101 to R1, R12 to R13, R13 to R14, R14 to R15, R11 to R16, R15 to R17, R102 to R2, R103 to R3, R104 to R4, R105 to R5, R4 to R6, R5 to R7, U101 to U1, U102 to U2, U103 to U3, Y101 to Y1
