File: key-matrix.kicad_sch (KiCad schematic)
At the start: 42 parts, among them J101 AudioJack4, J104 CONN_DISPLAY

Commit message: Add mounting holes
Parts:
- added H105, H106: MountingHole_Pad, MountingHole:MountingHole_2.2mm_M2_Pad_Via, symbol Mechanical:MountingHole_Pad
Connections:
- net GND: now also H105.1, H106.1
Other:
- moved on the sheet: H103, H104
Changed lines of the file:
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@@
     (stroke (width 0) (type default))
   )
-  (wire (pts (xy 54.864 125.984) (xy 54.864 124.968))
+  (wire (pts (xy 48.768 125.984) (xy 48.768 124.968))
     (stroke (width 0) (type default))
   )
@@
     (stroke (width 0) (type default))
   )
+  (wire (pts (xy 74.422 113.792) (xy 74.422 112.776))
+    (stroke (width 0) (type default))
+  )
   (wire (pts (xy 97.028 22.098) (xy 97.028 30.988))
     (stroke (width 0) (type default))
@@
     (stroke (width 0) (type default))
   )
+  (wire (pts (xy 74.168 127.254) (xy 74.168 126.238))
+    (stroke (width 0) (type default))
+  )
   (wire (pts (xy 159.258 38.608) (xy 169.418 38.608))
     (stroke (width 0) (type default))
@@
     (stroke (width 0) (type default))
   )
-  (wire (pts (xy 55.118 112.522) (xy 55.118 111.506))
+  (wire (pts (xy 49.022 112.522) (xy 49.022 111.506))
     (stroke (width 0) (type default))
   )
@@
     )
   )
-  (symbol (lib_name "GND_2") (lib_id "power:GND") (at 55.118 112.522 0) (unit 1)
-    (in_bom yes) (on_board yes) (dnp no) (fields_autoplaced)
-    (property "Reference" "#PWR0143" (at 55.118 118.872 0)
-      (effects (font (size 1.27 1.27)) hide)
-    )
-    (property "Value" "GND" (at 55.118 116.84 0)
-      (effects (font (size 1.27 1.27)))
-    )
-    (property "Footprint" "" (at 55.118 112.522 0)
-      (effects (font (size 1.27 1.27)) hide)
-    )
-    (property "Datasheet" "" (at 55.118 112.522 0)
+  (symbol (lib_name "GND_2") (lib_id "power:GND") (at 49.022 112.522 0) (unit 1)
+    (in_bom yes) (on_board yes) (dnp no) (fields_autoplaced)
+    (property "Reference" "#PWR0143" (at 49.022 118.872 0)
+      (effects (font (size 1.27 1.27)) hide)
+    )
+    (property "Value" "GND" (at 49.022 116.84 0)
+      (effects (font (size 1.27 1.27)))
+    )
+    (property "Footprint" "" (at 49.022 112.522 0)
+      (effects (font (size 1.27 1.27)) hide)
+    )
+    (property "Datasheet" "" (at 49.022 112.522 0)
       (effects (font (size 1.27 1.27)) hide)
     )
@@
     )
   )
+  (symbol (lib_id "Mechanical:MountingHole_Pad") (at 74.168 123.698 0) (unit 1)
+    (in_bom yes) (on_board yes) (dnp no) (fields_autoplaced)
+    (property "Reference" "H105" (at 77.47 121.158 0)
+      (effects (font (size 1.27 1.27)) (justify left))
+    )
+    (property "Value" "MountingHole_Pad" (at 77.47 123.698 0)
+      (effects (font (size 1.27 1.27)) (justify left))
+    )
+    (property "Footprint" "MountingHole:MountingHole_2.2mm_M2_Pad_Via" (at 74.168 123.698 0)
+      (effects (font (size 1.27 1.27)) hide)
+    )
+    (property "Datasheet" "~" (at 74.168 123.698 0)
+      (effects (font (size 1.27 1.27)) hide)
+    )
+    (pin "1")
+    (instances
+      (project "Interface"
+        (path "/c9f596c2-7857-4b11-bdf6-e9f4a0e624c2/fe52d998-1c79-453f-8784-76d0e74ea227"
+          (reference "H105") (unit 1)
+        )
+      )
+    )
+  )
   (symbol (lib_id "Switch:SW_Push") (at 84.328 46.228 0) (unit 1)
     (in_bom yes) (on_board yes) (dnp no) (fields_autoplaced)
@@
     )
   )
-  (symbol (lib_id "Mechanical:MountingHole_Pad") (at 55.118 108.966 0) (unit 1)
-    (in_bom yes) (on_board yes) (dnp no) (fields_autoplaced)
-    (property "Reference" "H103" (at 58.42 106.426 0)
-      (effects (font (size 1.27 1.27)) (justify left))
-    )
-    (property "Value" "MountingHole_Pad" (at 58.42 108.966 0)
-      (effects (font (size 1.27 1.27)) (justify left))
-    )
-    (property "Footprint" "MountingHole:MountingHole_2.2mm_M2_Pad_Via" (at 55.118 108.966 0)
-      (effects (font (size 1.27 1.27)) hide)
-    )
-    (property "Datasheet" "~" (at 55.118 108.966 0)
+  (symbol (lib_id "Mechanical:MountingHole_Pad") (at 49.022 108.966 0) (unit 1)
+    (in_bom yes) (on_board yes) (dnp no) (fields_autoplaced)
+    (property "Reference" "H103" (at 52.324 106.426 0)
+      (effects (font (size 1.27 1.27)) (justify left))
+    )
+    (property "Value" "MountingHole_Pad" (at 52.324 108.966 0)
+      (effects (font (size 1.27 1.27)) (justify left))
+    )
+    (property "Footprint" "MountingHole:MountingHole_2.2mm_M2_Pad_Via" (at 49.022 108.966 0)
+      (effects (font (size 1.27 1.27)) hide)
+    )
+    (property "Datasheet" "~" (at 49.022 108.966 0)
       (effects (font (size 1.27 1.27)) hide)
     )
@@
         (path "/c9f596c2-7857-4b11-bdf6-e9f4a0e624c2/fe52d998-1c79-453f-8784-76d0e74ea227"
           (reference "D105") (unit 1)
+        )
+      )
+    )
+  )
+  (symbol (lib_id "Mechanical:MountingHole_Pad") (at 74.422 110.236 0) (unit 1)
+    (in_bom yes) (on_board yes) (dnp no) (fields_autoplaced)
+    (property "Reference" "H106" (at 77.724 107.696 0)
+      (effects (font (size 1.27 1.27)) (justify left))
+    )
+    (property "Value" "MountingHole_Pad" (at 77.724 110.236 0)
+      (effects (font (size 1.27 1.27)) (justify left))
+    )
+    (property "Footprint" "MountingHole:MountingHole_2.2mm_M2_Pad_Via" (at 74.422 110.236 0)
+      (effects (font (size 1.27 1.27)) hide)
+    )
+    (property "Datasheet" "~" (at 74.422 110.236 0)
+      (effects (font (size 1.27 1.27)) hide)
+    )
+    (pin "1")
+    (instances
+      (project "Interface"
+        (path "/c9f596c2-7857-4b11-bdf6-e9f4a0e624c2/fe52d998-1c79-453f-8784-76d0e74ea227"
+          (reference "H106") (unit 1)
+        )
+      )
+    )
+  )
+  (symbol (lib_name "GND_2") (lib_id "power:GND") (at 74.422 113.792 0) (unit 1)
+    (in_bom yes) (on_board yes) (dnp no) (fields_autoplaced)
+    (property "Reference" "#PWR0155" (at 74.422 120.142 0)
+      (effects (font (size 1.27 1.27)) hide)
+    )
+    (property "Value" "GND" (at 74.422 118.11 0)
+      (effects (font (size 1.27 1.27)))
+    )
+    (property "Footprint" "" (at 74.422 113.792 0)
+      (effects (font (size 1.27 1.27)) hide)
+    )
+    (property "Datasheet" "" (at 74.422 113.792 0)
+      (effects (font (size 1.27 1.27)) hide)
+    )
+    (pin "1")
+    (instances
+      (project "Interface"
+        (path "/c9f596c2-7857-4b11-bdf6-e9f4a0e624c2/fe52d998-1c79-453f-8784-76d0e74ea227"
+          (reference "#PWR0155") (unit 1)
         )
       )
@@
     )
   )
-  (symbol (lib_id "Mechanical:MountingHole_Pad") (at 54.864 122.428 0) (unit 1)
-    (in_bom yes) (on_board yes) (dnp no) (fields_autoplaced)
-    (property "Reference" "H104" (at 58.166 119.888 0)
-      (effects (font (size 1.27 1.27)) (justify left))
-    )
-    (property "Value" "MountingHole_Pad" (at 58.166 122.428 0)
-      (effects (font (size 1.27 1.27)) (justify left))
-    )
-    (property "Footprint" "MountingHole:MountingHole_2.2mm_M2_Pad_Via" (at 54.864 122.428 0)
-      (effects (font (size 1.27 1.27)) hide)
-    )
-    (property "Datasheet" "~" (at 54.864 122.428 0)
+  (symbol (lib_id "Mechanical:MountingHole_Pad") (at 48.768 122.428 0) (unit 1)
+    (in_bom yes) (on_board yes) (dnp no) (fields_autoplaced)
+    (property "Reference" "H104" (at 52.07 119.888 0)
+      (effects (font (size 1.27 1.27)) (justify left))
+    )
+    (property "Value" "MountingHole_Pad" (at 52.07 122.428 0)
+      (effects (font (size 1.27 1.27)) (justify left))
+    )
+    (property "Footprint" "MountingHole:MountingHole_2.2mm_M2_Pad_Via" (at 48.768 122.428 0)
+      (effects (font (size 1.27 1.27)) hide)
+    )
+    (property "Datasheet" "~" (at 48.768 122.428 0)
       (effects (font (size 1.27 1.27)) hide)
     )
@@
         (path "/c9f596c2-7857-4b11-bdf6-e9f4a0e624c2/fe52d998-1c79-453f-8784-76d0e74ea227"
           (reference "MX109") (unit 1)
+        )
+      )
+    )
+  )
+  (symbol (lib_name "GND_2") (lib_id "power:GND") (at 74.168 127.254 0) (unit 1)
+    (in_bom yes) (on_board yes) (dnp no) (fields_autoplaced)
+    (property "Reference" "#PWR0121" (at 74.168 133.604 0)
+      (effects (font (size 1.27 1.27)) hide)
+    )
+    (property "Value" "GND" (at 74.168 131.572 0)
+      (effects (font (size 1.27 1.27)))
+    )
+    (property "Footprint" "" (at 74.168 127.254 0)
+      (effects (font (size 1.27 1.27)) hide)
+    )
+    (property "Datasheet" "" (at 74.168 127.254 0)
+      (effects (font (size 1.27 1.27)) hide)
+    )
+    (pin "1")
+    (instances
+      (project "Interface"
+        (path "/c9f596c2-7857-4b11-bdf6-e9f4a0e624c2/fe52d998-1c79-453f-8784-76d0e74ea227"
+          (reference "#PWR0121") (unit 1)
         )
       )
@@
     )
   )
-  (symbol (lib_name "GND_2") (lib_id "power:GND") (at 54.864 125.984 0) (unit 1)
-    (in_bom yes) (on_board yes) (dnp no) (fields_autoplaced)
-    (property "Reference" "#PWR0144" (at 54.864 132.334 0)
-      (effects (font (size 1.27 1.27)) hide)
-    )
-    (property "Value" "GND" (at 54.864 130.302 0)
-      (effects (font (size 1.27 1.27)))
-    )
-    (property "Footprint" "" (at 54.864 125.984 0)
-      (effects (font (size 1.27 1.27)) hide)
-    )
-    (property "Datasheet" "" (at 54.864 125.984 0)
-      (effects (font (size 1.27 1.27)) hide)
-    )
+  (symbol (lib_name "GND_2") (lib_id "power:GND") (at 48.768 125.984 0) (unit 1)
+    (in_bom yes) (on_board yes) (dnp no) (fields_autoplaced)
+    (property "Reference" "#PWR0144" (at 48.768 132.334 0)
+      (effects (font (size 1.27 1.27)) hide)
+    )
+    (property "Value" "GND" (at 48.768 130.302 0)
+      (effects (font (size 1.27 1.27)))
+    )
+    (property "Footprint" "" (at 48.768 125.984 0)
+      (effects (font (size 1.27 1.27)) hide)
+    )
+    (property "Datasheet" "" (at 48.768 125.984 0)
+      (effects (font (size 1.27 1.27)) hide)
+    )

Commit message: Cleanup routing
Parts:
- H101, H102, H103, H104, H105, H106: footprint MountingHole:MountingHole_2.2mm_M2_Pad_Via -> MountingHole:MountingHole_2.2mm_M2_Pad
Changed lines of the file:
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@@
       (effects (font (size 1.27 1.27)) (justify left))
     )
-    (property "Footprint" "MountingHole:MountingHole_2.2mm_M2_Pad_Via" (at 22.606 108.712 0)
+    (property "Footprint" "MountingHole:MountingHole_2.2mm_M2_Pad" (at 22.606 108.712 0)
       (effects (font (size 1.27 1.27)) hide)
     )
@@
       (effects (font (size 1.27 1.27)) (justify left))
     )
-    (property "Footprint" "MountingHole:MountingHole_2.2mm_M2_Pad_Via" (at 74.168 123.698 0)
+    (property "Footprint" "MountingHole:MountingHole_2.2mm_M2_Pad" (at 74.168 123.698 0)
       (effects (font (size 1.27 1.27)) hide)
     )
@@
       (effects (font (size 1.27 1.27)) (justify left))
     )
-    (property "Footprint" "MountingHole:MountingHole_2.2mm_M2_Pad_Via" (at 49.022 108.966 0)
+    (property "Footprint" "MountingHole:MountingHole_2.2mm_M2_Pad" (at 49.022 108.966 0)
       (effects (font (size 1.27 1.27)) hide)
     )
@@
       (effects (font (size 1.27 1.27)) (justify left))
     )
-    (property "Footprint" "MountingHole:MountingHole_2.2mm_M2_Pad_Via" (at 74.422 110.236 0)
+    (property "Footprint" "MountingHole:MountingHole_2.2mm_M2_Pad" (at 74.422 110.236 0)
       (effects (font (size 1.27 1.27)) hide)
     )
@@
       (effects (font (size 1.27 1.27)) (justify left))
     )
-    (property "Footprint" "MountingHole:MountingHole_2.2mm_M2_Pad_Via" (at 48.768 122.428 0)
+    (property "Footprint" "MountingHole:MountingHole_2.2mm_M2_Pad" (at 48.768 122.428 0)
       (effects (font (size 1.27 1.27)) hide)
     )
@@
       (effects (font (size 1.27 1.27)) (justify left))
     )
-    (property "Footprint" "MountingHole:MountingHole_2.2mm_M2_Pad_Via" (at 22.606 122.682 0)
-      (effects (font (size 1.27 1.27)) hide)
-    )
+    (property "Footprint" "MountingHole:MountingHole_2.2mm_M2_Pad" (at 22.606 122.682 0)
+      (effects (font (size 1.27 1.27)) hide)
+    )

Commit message: Rotate and add mirror line
Parts:
- renumbered D103 to D101, D104 to D102, D105 to D103, D106 to D104, D107 to D105, D108 to D106, D109 to D107, D110 to D108, D111 to D109, D112 to D110, D113 to D111, D114 to D112, D115 to D113, D116 to D114, D117 to D115, D118 to D116, D119 to D117, J104 to J4
